Commit message: fix wheel link

File: amr_ws/install/robot_description/share/robot_description/urdf/caster_ball.xacro (robot description, xacro)
@@ -1,33 +1,5 @@
-<?xml version='1.0'?>
-<robot name="robot" xmlns:xacro="http://www.ros.org/wiki/xacro">
-  <xacro:include filename="$(find robot_description)/urdf/differential_robot.gazebo" />
-  <xacro:include filename="$(find robot_description)/urdf/materials.xacro" />
-  <xacro:include filename="$(find robot_description)/urdf/xacro_variables.xacro" />
-  <xacro:include filename="$(find robot_description)/urdf/wheels.xacro" />
-  <xacro:include filename="$(find robot_description)/urdf/caster_ball.xacro" />
-  <link name='chassis'>
-    <pose>0 0 0.1 0 0 0</pose>
-    <inertial>
-      <mass value="10.0"/>
-      <origin xyz="0.0 0 0.1" rpy=" 0 0 0"/>
-      <cylinder_inertia m="10" r="${chasis_cylinder_radius}" h="${chasis_cylinder_height}"/>
-      <inertia
-          ixx="0.5" ixy="0" ixz="0"
-          iyy="1.0" iyz="0"
-          izz="0.1"
-      />
-    </inertial>
-    <collision name='collision'>
-      <geometry>
-        <cylinder radius="${chasis_cylinder_radius}" length="${chasis_cylinder_height}"/>
-      </geometry>
-    </collision>
-    <visual name='chassis_visual'>
-      <origin xyz="0 0 0" rpy=" 0 0 0"/>
-      <geometry>
-        <cylinder radius="${chasis_cylinder_radius}" length="${chasis_cylinder_height}"/>
-      </geometry>
-      <material name="blue"/>
-    </visual>
+<?xml version="1.0"?>
+<robot xmlns:xacro="http://www.ros.org/wiki/xacro">
+  <xacro:macro name="caster_balls_macro">
     <collision name='caster_collision'>
       <origin xyz="${chasis_caster_x} ${chasis_caster_y} ${chasis_caster_z}" rpy=" ${chasis_caster_r} ${chasis_caster_p} ${chasis_caster_ya}"/>
@@ -76,7 +48,4 @@
       <material name="orange"/>
     </visual>
-  </link>
-  <!-- Include wheel and caster macros -->
-  <xacro:wheels_macro />
-  <xacro:caster_balls_macro />
+  </xacro:macro>
 </robot>
