Commit message: APS 2 working

File: amr_ws/install/robot_description/share/robot_description/urdf/xacro_variables.xacro (robot description, xacro)
@@ -3,7 +3,8 @@
 <!--Xacro variable declaration-->
 <!--Dimentions-->
-  <!--Chasis_cylinder-->
-  <xacro:property name="chasis_cylinder_radius" value="0.2" />
-  <xacro:property name="chasis_cylinder_height" value="0.05" />
+  <!--Chasis_box-->
+  <xacro:property name="chasis_box_length" value="0.4" />
+  <xacro:property name="chasis_box_width" value="0.3" />
+  <xacro:property name="chasis_box_height" value="0.15" />
   <!--Chasis_caster-->
   <xacro:property name="chasis_caster_radius" value="0.05" />
@@ -12,11 +13,11 @@
   <xacro:property name="wheel_cylinder_height" value="0.05" />
 <!--Positions-->
-  <!--Chasis_cylinder-->
-  <xacro:property name="chasis_cylinder_x" value="0" />
-  <xacro:property name="chasis_cylinder_y" value="0" />
-  <xacro:property name="chasis_cylinder_z" value="0.1" />
-  <xacro:property name="chasis_cylinder_r" value="0" />
-  <xacro:property name="chasis_cylinder_p" value="0" />
-  <xacro:property name="chasis_cylinder_ya" value="0" />
+  <!--Chasis_box-->
+  <xacro:property name="chasis_box_x" value="0" />
+  <xacro:property name="chasis_box_y" value="0" />
+  <xacro:property name="chasis_box_z" value="0.15" />
+  <xacro:property name="chasis_box_r" value="0" />
+  <xacro:property name="chasis_box_p" value="0" />
+  <xacro:property name="chasis_box_ya" value="0" />
   <!--Chasis_caster-->
   <xacro:property name="chasis_caster_x" value="-0.15" />
