Commit message: fixed robot_description.launch.py

File: amr_ws/src/robot_description/urdf/differential_robot.xacro (robot description, xacro)
@@ -6,4 +6,12 @@
   <xacro:include filename="$(find robot_description)/urdf/wheels.xacro" />
   <xacro:include filename="$(find robot_description)/urdf/caster_ball.xacro" />
+  <!-- Add dummy base link -->
+  <link name="base_link">
+  </link>
+  <joint name="base_joint" type="fixed">
+    <parent link="base_link"/>
+    <child link="chassis"/>
+    <origin xyz="0 0 0" rpy="0 0 0"/>
+  </joint>
   <link name='chassis'>
     <pose>0 0 0.1 0 0 0</pose>
@@ -11,5 +19,5 @@
       <mass value="10.0"/>
       <origin xyz="0.0 0 0.1" rpy=" 0 0 0"/>
-      <cylinder_inertia m="10" r="${chasis_cylinder_radius}" h="${chasis_cylinder_height}"/>
+      <box_inertia m="10" l="${chasis_box_length}" w="${chasis_box_width}" h="${chasis_box_height}"/>
       <inertia
           ixx="0.5" ixy="0" ixz="0"
@@ -20,5 +28,5 @@
     <collision name='collision'>
       <geometry>
-        <cylinder radius="${chasis_cylinder_radius}" length="${chasis_cylinder_height}"/>
+        <box size="${chasis_box_length} ${chasis_box_width} ${chasis_box_height}"/>
       </geometry>
     </collision>
@@ -26,7 +34,7 @@
       <origin xyz="0 0 0" rpy=" 0 0 0"/>
       <geometry>
-        <cylinder radius="${chasis_cylinder_radius}" length="${chasis_cylinder_height}"/>
+        <box size="${chasis_box_length} ${chasis_box_width} ${chasis_box_height}"/>
       </geometry>
-      <material name="blue"/>
+      <material name="red"/>
     </visual>
     <collision name='caster_collision'>

File: amr_ws/src/robot_description/urdf/xacro_variables.xacro (robot description, xacro)
@@ -3,7 +3,8 @@
 <!--Xacro variable declaration-->
 <!--Dimentions-->
-  <!--Chasis_cylinder-->
-  <xacro:property name="chasis_cylinder_radius" value="0.2" />
-  <xacro:property name="chasis_cylinder_height" value="0.05" />
+  <!--Chasis_box-->
+  <xacro:property name="chasis_box_length" value="0.4" />
+  <xacro:property name="chasis_box_width" value="0.3" />
+  <xacro:property name="chasis_box_height" value="0.1" />
   <!--Chasis_caster-->
   <xacro:property name="chasis_caster_radius" value="0.05" />
@@ -12,11 +13,11 @@
   <xacro:property name="wheel_cylinder_height" value="0.05" />
 <!--Positions-->
-  <!--Chasis_cylinder-->
-  <xacro:property name="chasis_cylinder_x" value="0" />
-  <xacro:property name="chasis_cylinder_y" value="0" />
-  <xacro:property name="chasis_cylinder_z" value="0.1" />
-  <xacro:property name="chasis_cylinder_r" value="0" />
-  <xacro:property name="chasis_cylinder_p" value="0" />
-  <xacro:property name="chasis_cylinder_ya" value="0" />
+  <!--Chasis_box-->
+  <xacro:property name="chasis_box_x" value="0" />
+  <xacro:property name="chasis_box_y" value="0" />
+  <xacro:property name="chasis_box_z" value="0.1" />
+  <xacro:property name="chasis_box_r" value="0" />
+  <xacro:property name="chasis_box_p" value="0" />
+  <xacro:property name="chasis_box_ya" value="0" />
   <!--Chasis_caster-->
   <xacro:property name="chasis_caster_x" value="-0.15" />
