Commit message: project 1 complete

File: amr_ws/src/robot_description/urdf/robot_base.xacro (robot description, xacro)
@@ -1,17 +1,13 @@
 <?xml version='1.0'?>
 <robot name="robot" xmlns:xacro="http://www.ros.org/wiki/xacro">
-  <xacro:include filename="$(find robot_description)/urdf/differential_robot.gazebo" />
+  <xacro:include filename="$(find robot_description)/urdf/robot_base.gazebo" />
   <xacro:include filename="$(find robot_description)/urdf/materials.xacro" />
   <xacro:include filename="$(find robot_description)/urdf/xacro_variables.xacro" />
   <xacro:include filename="$(find robot_description)/urdf/wheels.xacro" />
   <xacro:include filename="$(find robot_description)/urdf/caster_ball.xacro" />
+  <xacro:include filename="$(find robot_description)/urdf/sensors.xacro" />
   <!-- Add dummy base link -->
   <link name="base_link">
   </link>
-  <joint name="base_joint" type="fixed">
-    <parent link="base_link"/>
-    <child link="chassis"/>
-    <origin xyz="0 0 0" rpy="0 0 0"/>
-  </joint>
   <link name='chassis'>
     <pose>0 0 0.1 0 0 0</pose>
@@ -85,4 +81,42 @@
     </visual>
   </link>
+  <joint name="base_joint" type="fixed">
+    <parent link="base_link"/>
+    <child link="chassis"/>
+    <origin xyz="0 0 0" rpy="0 0 0"/>
+  </joint>
+  <link name="imu_link">
+  </link>
+  <joint name="imu_joint" type="fixed">
+    <parent link="chassis"/>
+    <child link="imu_link"/>
+    <origin xyz="0 0 0" rpy="0 0 0"/>
+  </joint>
+  <link name="lidar_link">
+    <visual name="lidar_visual">
+      <origin xyz="0 0 0.07" rpy="0 0 0"/>
+      <geometry>
+        <cylinder radius="0.1" length="0.05"/>
+      </geometry>
+    </visual>
+  </link>
+  <joint name="lidar_joint" type="fixed">
+    <parent link="chassis"/>
+    <child link="lidar_link"/>
+    <origin xyz="0 0 0.07" rpy="0 0 0"/>
+  </joint>
+  <link name="camera_link">
+    <visual name="camera_visual">
+      <origin xyz="0.11 0 0" rpy="0 0 0"/>
+      <geometry>
+        <box size="0.02 0.15 0.1"/>
+      </geometry>
+    </visual>
+  </link>
+  <joint name="camera_joint" type="fixed">
+    <parent link="chassis"/>
+    <child link="camera_link"/>
+    <origin xyz="0.11 0 0" rpy="0 0 0"/>
+  </joint>
   <!-- Include wheel and caster macros -->
   <xacro:wheels_macro />

File: amr_ws/src/robot_description/urdf/sensors.xacro (robot description, xacro)
@@ -1,92 +1,93 @@
-<!-- IMU Plugin -->
-<gazebo>
-  <sensor name="my_imu" type="imu">
-    <always_on>true</always_on>
-    <update_rate>30</update_rate>
-    <topic>imu</topic>
-    <gaussian_noise>0.001 0.001 0.001</gaussian_noise>
-    <plugin name="imu_plugin" filename="libgazebo_ros_imu_sensor.so">
-      <ros>
-        <namespace>imu_sensor</namespace>
-        <remapping>
-          <imu>imu</imu>
-        </remapping>
-      </ros>
-    </plugin>
-  </sensor>
-</gazebo>
-<!-- Lidar Plugin -->
-<gazebo reference="lidar_link">
-    <sensor name="laser" type="ray">
-        <pose>0 0 0 0 0 0</pose>
-        <visualize>true</visualize>
+<?xml version='1.0'?>
+<robot name="robot" xmlns:xacro="http://www.ros.org/wiki/xacro">
+    <!-- IMU Plugin -->
+    <gazebo reference="imu_link">
+    <sensor name="imu" type="imu">
+        <always_on>true</always_on>
         <update_rate>10</update_rate>
-        <topic>lidar_scan</topic>
-        <ray>
-            <scan>
-                <horizontal>
-                    <samples>720</samples>
-                    <resolution>1</resolution>
-                    <min_angle>-3.14159</min_angle>
-                    <max_angle>3.14159</max_angle>
-                </horizontal>
-            </scan>
-            <range>
-                <min>0.1</min>
-                <max>100.0</max>
-            </range>
-        </ray>
-        <plugin name="laser_controller" filename="libgazebo_ros_ray_sensor.so">
+        <plugin name="imu_plugin" filename="libgazebo_ros_imu_sensor.so">
+            <frame_name>imu_link</frame_name>
             <ros>
-                <argument>~/out:=scan</argument>
+                <remapping>~/out:=/imu/data</remapping>
             </ros>
-            <output_type>sensor_msgs/LaserScan</output_type>
-            <frame_name>lidar_link</frame_name>
         </plugin>
     </sensor>
-</gazebo>
-<!-- Camera Plugin -->
-<gazebo reference="camera_link">
-    <sensor name="camera" type="camera">
-        <pose>0 0 0 0 0 0</pose>
-        <visualize>true</visualize>
-        <update_rate>10</update_rate>
-        <camera>
-            <horizontal_fov>1.089</horizontal_fov>
-            <image>
-                <format>R8G8B8</format>
-                <width>640</width>
-                <height>480</height>
-            </image>
-            <clip>
-                <near>0.05</near>
-                <far>8.0</far>
-            </clip>
-        </camera>
-        <plugin name="camera_controller" filename="libgazebo_ros_camera.so">
-            <frame_name>camera_link</frame_name>
+    </gazebo>
+    <!-- Lidar Plugin -->
+    <gazebo reference="lidar_link">
+        <sensor name="laser" type="ray">
+            <pose>0 0 0.07 0 0 0</pose>
+            <visualize>true</visualize>
+            <update_rate>10</update_rate>
+            <ray>
+                <scan>
+                    <horizontal>
+                        <samples>720</samples>
+                        <resolution>1</resolution>
+                        <min_angle>-3.14159</min_angle>
+                        <max_angle>3.14159</max_angle>
+                    </horizontal>
+                </scan>
+                <range>
+                    <min>0.1</min>
+                    <max>10</max>
+                    <resolution>0.015000</resolution>
+                </range>
+                <noise>
+                    <type>gaussian</type>
+                    <mean>0.0</mean>
+                    <stddev>0.01</stddev>
+                </noise>
+            </ray>
+            <plugin name="laser_controller" filename="libgazebo_ros_ray_sensor.so">
+                <output_type>sensor_msgs/LaserScan</output_type>
+                <frame_name>lidar_link</frame_name>
+                <ros>
+                    <remapping>~/out:=/scan</remapping>
+                </ros>
+            </plugin>
+        </sensor>
+    </gazebo>
+    <!-- Camera Plugin -->
+    <gazebo reference="camera_link">
+        <sensor name="camera" type="camera">
+            <pose>0.11 0 0 0 0 0</pose>
+            <visualize>true</visualize>
+            <update_rate>10</update_rate>
+            <image_topic_name>camera/image_raw</image_topic_name>
+            <camera_info_topic_name>camera/camera_info</camera_info_topic_name>
+            <camera>
+                <horizontal_fov>1.089</horizontal_fov>
+                <image>
+                    <format>R8G8B8</format>
+                    <width>640</width>
+                    <height>480</height>
+                </image>
+                <clip>
+                    <near>0.05</near>
+                    <far>8.0</far>
+                </clip>
+            </camera>
+            <plugin name="camera_controller" filename="libgazebo_ros_camera.so">
+                <frame_name>camera_link</frame_name>
+            </plugin>
+        </sensor>
+    </gazebo>
+    <!-- Differential Controller Plugin -->
+    <gazebo>
+        <plugin name="gazebo_ros_diff_drive" filename="libgazebo_ros_diff_drive.so">
+            <update_rate>10</update_rate>
+            <left_joint>left_wheel_hinge</left_joint>
+            <right_joint>right_wheel_hinge</right_joint>
+            <wheel_separation>0.4</wheel_separation>
+            <wheel_diameter>0.2</wheel_diameter>
+            <command_topic>cmd_vel</command_topic>
+            <publish_odom>true</publish_odom>
+            <publish_odom_tf>true</publish_odom_tf>
+            <publish_wheel_tf>true</publish_wheel_tf>
+            <odometry_topic>odom</odometry_topic>
+            <odometry_frame>odom</odometry_frame>
+            <robot_base_frame>base_link</robot_base_frame>
         </plugin>
-    </sensor>
-</gazebo>
-<!-- Differential Controller Plugin -->
-<gazebo>
-    <plugin name="gazebo_ros_diff_drive" filename="libgazebo_ros_diff_drive.so">
-        <ros>
-            <namespace>diff_drive_controller</namespace>
-        </ros>
-        <update_rate>50</update_rate>
-        <left_joint>left_wheel_joint</left_joint>
-        <right_joint>right_wheel_joint</right_joint>
-        <wheel_separation>0.4</wheel_separation>
-        <wheel_diameter>0.2</wheel_diameter>
-        <max_wheel_torque>200</max_wheel_torque>
-        <max_wheel_acceleration>5</max_wheel_acceleration>
-        <command_topic>cmd_vel</command_topic>
-        <publish_odom>true</publish_odom>
-        <publish_odom_tf>true</publish_odom_tf>
-        <publish_wheel_tf>true</publish_wheel_tf>
-        <odometry_topic>odom</odometry_topic>
-        <odometry_frame>odom</odometry_frame>
-        <robot_base_frame>chassis</robot_base_frame>
-    </plugin>
-</gazebo>
+    </gazebo>
+</robot>

File: amr_ws/src/robot_description/urdf/wheels.xacro (robot description, xacro)
@@ -53,7 +53,6 @@
       <origin xyz="${left_wheel_x} ${left_wheel_y} ${left_wheel_z}" rpy="0 0 0"/>
       <child link="left_wheel"/>
-      <parent link="chassis"/>
+      <parent link="base_link"/>
       <axis xyz="0 1 0" rpy="0 0 0"/>
-      <limit effort="100" velocity="100"/>
       <joint_properties damping="0.0" friction="0.0"/>
     </joint>
@@ -61,7 +60,6 @@
       <origin xyz="${right_wheel_x} ${right_wheel_y} ${right_wheel_z}" rpy="0 0 0"/>
       <child link="right_wheel"/>
-      <parent link="chassis"/>
+      <parent link="base_link"/>
       <axis xyz="0 1 0" rpy="0 0 0"/>
-      <limit effort="100" velocity="100"/>
       <joint_properties damping="0.0" friction="0.0"/>
     </joint>

File: amr_ws/src/robot_description/urdf/xacro_variables.xacro (robot description, xacro)
@@ -6,5 +6,5 @@
   <xacro:property name="chasis_box_length" value="0.4" />
   <xacro:property name="chasis_box_width" value="0.3" />
-  <xacro:property name="chasis_box_height" value="0.1" />
+  <xacro:property name="chasis_box_height" value="0.15" />
   <!--Chasis_caster-->
   <xacro:property name="chasis_caster_radius" value="0.05" />
@@ -16,5 +16,5 @@
   <xacro:property name="chasis_box_x" value="0" />
   <xacro:property name="chasis_box_y" value="0" />
-  <xacro:property name="chasis_box_z" value="0.1" />
+  <xacro:property name="chasis_box_z" value="0.15" />
   <xacro:property name="chasis_box_r" value="0" />
   <xacro:property name="chasis_box_p" value="0" />
